Commit message: quadruped + stuff

File: body.urdf (robot description, URDF)
Before this commit: robot robot, 3 links, 2 joints
Links:
- added link BackLeg2, mass 1; collision box size=0.2 0.2 1; visual box size=0.2 0.2 1
- added link FrontLeg2, mass 1; collision box size=0.2 0.2 1; visual box size=0.2 0.2 1
- added link LeftLeg, mass 1; collision box size=1 0.2 0.2; visual box size=1 0.2 0.2
- added link LeftLeg2, mass 1; collision box size=0.2 0.2 1; visual box size=0.2 0.2 1
- added link RightLeg, mass 1; collision box size=1 0.2 0.2; visual box size=1 0.2 0.2
- added link RightLeg2, mass 1; collision box size=0.2 0.2 1; visual box size=0.2 0.2 1
- link BackLeg: geometry collision box size=0.2 1 0.2; visual box size=0.2 1 0.2
- link FrontLeg: geometry collision box size=0.2 1 0.2; visual box size=0.2 1 0.2
Joints:
- added joint BackLeg_BackLeg2: type revolute, parent BackLeg, child BackLeg2, origin xyz=0 -1 0 rpy=0 0 0, axis 1 0 0, limit lower=-3.14159 upper=3.14159 effort=0.0 velocity=0.0
- added joint FrontLeg_FrontLeg2: type revolute, parent FrontLeg, child FrontLeg2, origin xyz=0 1 0 rpy=0 0 0, axis 1 0 0, limit lower=-3.14159 upper=3.14159 effort=0.0 velocity=0.0
- added joint LeftLeg_LeftLeg2: type revolute, parent LeftLeg, child LeftLeg2, origin xyz=-1 0 0 rpy=0 0 0, axis 0 1 0, limit lower=-3.14159 upper=3.14159 effort=0.0 velocity=0.0
- added joint RightLeg_RightLeg2: type revolute, parent RightLeg, child RightLeg2, origin xyz=1 0 0 rpy=0 0 0, axis 0 1 0, limit lower=-3.14159 upper=3.14159 effort=0.0 velocity=0.0
- added joint Torso_LeftLeg: type revolute, parent Torso, child LeftLeg, origin xyz=-0.5 0 1 rpy=0 0 0, axis 0 1 0, limit lower=-3.14159 upper=3.14159 effort=0.0 velocity=0.0
- added joint Torso_RightLeg: type revolute, parent Torso, child RightLeg, origin xyz=0.5 0 1 rpy=0 0 0, axis 0 1 0, limit lower=-3.14159 upper=3.14159 effort=0.0 velocity=0.0
- joint Torso_BackLeg: axis 0 1 0 -> 1 0 0; origin xyz=-0.5 0 1 rpy=0 0 0 -> xyz=0 -0.5 1 rpy=0 0 0
- joint Torso_FrontLeg: axis 0 1 0 -> 1 0 0; origin xyz=0.5 0 1 rpy=0 0 0 -> xyz=0 0.5 1 rpy=0 0 0

Commit message: temp

File: body.urdf (robot description, URDF)
Before this commit: robot robot, 9 links, 8 joints
Links:
- removed link BackLeg
- removed link BackLeg2
- removed link FrontLeg
- removed link FrontLeg2
- removed link LeftLeg
- removed link LeftLeg2
- removed link RightLeg
- removed link RightLeg2
- added link Abdomen, mass 1; collision box size=0.5 0.6 0.5; visual box size=0.5 0.6 0.5
- link Torso: geometry collision box size=0.75 0.5 0.4; visual box size=0.75 0.5 0.4
Joints:
- removed joint BackLeg_BackLeg2
- removed joint FrontLeg_FrontLeg2
- removed joint LeftLeg_LeftLeg2
- removed joint RightLeg_RightLeg2
- removed joint Torso_BackLeg
- removed joint Torso_FrontLeg
- removed joint Torso_LeftLeg
- removed joint Torso_RightLeg
- added joint Torso_Abdomen: type revolute, parent Torso, child Abdomen, origin xyz=0 0 0.75 rpy=0 0 0, axis 1 0 0, limit lower=-3.14159 upper=3.14159 effort=0.0 velocity=0.0

Commit message: assignemtn 5

File: body.urdf (robot description, URDF)
Before this commit: robot robot, 2 links, 1 joints
Links:
- added link Head, mass 1; collision box size=0.75 0.4 0.3; visual box size=0.75 0.4 0.3
- added link LBLeg1, mass 1; collision box size=0.2 0.75 0.2; visual box size=0.2 0.75 0.2
- added link LBLeg2, mass 1; collision box size=0.2 0.2 0.75; visual box size=0.2 0.2 0.75
- added link LFLeg1, mass 1; collision box size=0.2 0.75 0.2; visual box size=0.2 0.75 0.2
- added link LFLeg2, mass 1; collision box size=0.2 0.2 0.75; visual box size=0.2 0.2 0.75
- added link LMLeg1, mass 1; collision box size=0.2 0.75 0.2; visual box size=0.2 0.75 0.2
- added link LMLeg2, mass 1; collision box size=0.2 0.2 0.75; visual box size=0.2 0.2 0.75
- added link RBLeg1, mass 1; collision box size=0.2 0.75 0.2; visual box size=0.2 0.75 0.2
- added link RBLeg2, mass 1; collision box size=0.2 0.2 0.75; visual box size=0.2 0.2 0.75
- added link RFLeg1, mass 1; collision box size=0.2 0.75 0.2; visual box size=0.2 0.75 0.2
- added link RFLeg2, mass 1; collision box size=0.2 0.2 0.75; visual box size=0.2 0.2 0.75
- added link RMLeg1, mass 1; collision box size=0.2 0.75 0.2; visual box size=0.2 0.75 0.2
- added link RMLeg2, mass 1; collision box size=0.2 0.2 0.75; visual box size=0.2 0.2 0.75
- link Abdomen: geometry collision box size=0.75 0.4 0.3; visual box size=0.75 0.4 0.3
- link Torso: geometry collision box size=0.75 0.4 0.3; visual box size=0.75 0.4 0.3
Joints:
- added joint Abdomen_LBLeg1: type revolute, parent Abdomen, child LBLeg1, origin xyz=0.65 0.2 0 rpy=0 0 0, axis 1 0 -1, limit lower=-3.14159 upper=3.14159 effort=0.0 velocity=0.0
- added joint Abdomen_RBLeg1: type revolute, parent Abdomen, child RBLeg1, origin xyz=0.65 -0.2 0 rpy=0 0 0, axis 1 0 -1, limit lower=-3.14159 upper=3.14159 effort=0.0 velocity=0.0
- added joint Head_LFLeg1: type revolute, parent Head, child LFLeg1, origin xyz=-0.65 0.2 0 rpy=0 0 0, axis 1 0 1, limit lower=-3.14159 upper=3.14159 effort=0.0 velocity=0.0
- added joint Head_RFLeg1: type revolute, parent Head, child RFLeg1, origin xyz=-0.65 -0.2 0 rpy=0 0 0, axis 1 0 1, limit lower=-3.14159 upper=3.14159 effort=0.0 velocity=0.0
- added joint LBLeg1_LBLeg2: type revolute, parent LBLeg1, child LBLeg2, origin xyz=0 0.75 0 rpy=0 0 0, axis 1 0 0, limit lower=-3.14159 upper=3.14159 effort=0.0 velocity=0.0
- added joint LFLeg1_LFLeg2: type revolute, parent LFLeg1, child LFLeg2, origin xyz=0 0.75 0 rpy=0 0 0, axis 1 0 0, limit lower=-3.14159 upper=3.14159 effort=0.0 velocity=0.0
- added joint LMLeg1_LMLeg2: type revolute, parent LMLeg1, child LMLeg2, origin xyz=0 0.75 0 rpy=0 0 0, axis 1 0 0, limit lower=-3.14159 upper=3.14159 effort=0.0 velocity=0.0
- added joint RBLeg1_RBLeg2: type revolute, parent RBLeg1, child RBLeg2, origin xyz=0 -0.75 0 rpy=0 0 0, axis 1 0 0, limit lower=-3.14159 upper=3.14159 effort=0.0 velocity=0.0
- added joint RFLeg1_RFLeg2: type revolute, parent RFLeg1, child RFLeg2, origin xyz=0 -0.75 0 rpy=0 0 0, axis 1 0 0, limit lower=-3.14159 upper=3.14159 effort=0.0 velocity=0.0
- added joint RMLeg1_RMLeg2: type revolute, parent RMLeg1, child RMLeg2, origin xyz=0 -0.75 0 rpy=0 0 0, axis 1 0 0, limit lower=-3.14159 upper=3.14159 effort=0.0 velocity=0.0
- added joint Torso_Head: type revolute, parent Torso, child Head, origin xyz=-0.375 0 1 rpy=0 0 0, axis 0 0 1, limit lower=-3.14159 upper=3.14159 effort=0.0 velocity=0.0
- added joint Torso_LMLeg1: type revolute, parent Torso, child LMLeg1, origin xyz=0 0.2 1 rpy=0 0 0, axis 1 0 1, limit lower=-3.14159 upper=3.14159 effort=0.0 velocity=0.0
- added joint Torso_RMLeg1: type revolute, parent Torso, child RMLeg1, origin xyz=0 -0.2 1 rpy=0 0 0, axis 1 0 1, limit lower=-3.14159 upper=3.14159 effort=0.0 velocity=0.0
- joint Torso_Abdomen: axis 1 0 0 -> 0 0 1; origin xyz=0 0 0.75 rpy=0 0 0 -> xyz=0.375 0 1 rpy=0 0 0

Commit message: fin

File: body.urdf (robot description, URDF)
Before this commit: robot robot, 15 links, 14 joints
Links:
- removed link LMLeg1
- removed link LMLeg2
- removed link RMLeg1
- removed link RMLeg2
Joints:
- removed joint LMLeg1_LMLeg2
- removed joint RMLeg1_RMLeg2
- removed joint Torso_LMLeg1
- removed joint Torso_RMLeg1
- joint Abdomen_LBLeg1: origin xyz=0.65 0.2 0 rpy=0 0 0 -> xyz=0.65 0.2 0 rpy=0 0 -45
- joint Abdomen_RBLeg1: axis 1 0 -1 -> 1 0 1; origin xyz=0.65 -0.2 0 rpy=0 0 0 -> xyz=0.65 -0.2 0 rpy=0 0 45
- joint Head_LFLeg1: axis 1 0 1 -> 1 0 -1; origin xyz=-0.65 0.2 0 rpy=0 0 0 -> xyz=-0.65 0.2 0 rpy=0 0 45
- joint Head_RFLeg1: origin xyz=-0.65 -0.2 0 rpy=0 0 0 -> xyz=-0.65 -0.2 0 rpy=0 0 -45
- joint LBLeg1_LBLeg2: axis 1 0 0 -> 1 0 -1
- joint LFLeg1_LFLeg2: axis 1 0 0 -> 1 0 -1
- joint RBLeg1_RBLeg2: axis 1 0 0 -> 1 0 1
- joint RFLeg1_RFLeg2: axis 1 0 0 -> 1 0 1
- joint Torso_Abdomen: axis 0 0 1 -> 0 1 0
- joint Torso_Head: axis 0 0 1 -> 0 1 0

Commit message: snake

File: body.urdf (robot description, URDF)
Before this commit: robot robot, 11 links, 10 joints
Links:
- removed link Abdomen
- removed link Head
- removed link LBLeg1
- removed link LBLeg2
- removed link LFLeg1
- removed link LFLeg2
- removed link RBLeg1
- removed link RBLeg2
- removed link RFLeg1
- removed link RFLeg2
- removed link Torso
- added link 1, mass 1; collision box size=0.7174537699741859 0.686825274564822 1.1081465627597216; visual box size=0.7174537699741859 0.686825274564822 1.1081465627597216
- added link 2, mass 1; collision box size=1.4143638648991648 0.16316232412654819 1.368785566737274; visual box size=1.4143638648991648 0.16316232412654819 1.368785566737274
- added link 3, mass 1; collision box size=1.0538674862453004 0.2544337823310324 0.4878990057576473; visual box size=1.0538674862453004 0.2544337823310324 0.4878990057576473
- added link 4, mass 1; collision box size=0.3793270408250468 1.5490392038465357 0.6847540923456942; visual box size=0.3793270408250468 1.5490392038465357 0.6847540923456942
Joints:
- removed joint Abdomen_LBLeg1
- removed joint Abdomen_RBLeg1
- removed joint Head_LFLeg1
- removed joint Head_RFLeg1
- removed joint LBLeg1_LBLeg2
- removed joint LFLeg1_LFLeg2
- removed joint RBLeg1_RBLeg2
- removed joint RFLeg1_RFLeg2
- removed joint Torso_Abdomen
- removed joint Torso_Head
- added joint 1_2: type revolute, parent 1, child 2, origin xyz=-0.35872688498709293 0 1 rpy=0 0 0, axis 0 1 0, limit lower=-3.14159 upper=3.14159 effort=0.0 velocity=0.0
- added joint 1_3: type revolute, parent 1, child 3, origin xyz=0.35872688498709293 0 1 rpy=0 0 0, axis 0 1 0, limit lower=-3.14159 upper=3.14159 effort=0.0 velocity=0.0
- added joint 3_4: type revolute, parent 3, child 4, origin xyz=1.0538674862453004 0 0 rpy=0 0 0, axis 0 1 0, limit lower=-3.14159 upper=3.14159 effort=0.0 velocity=0.0

Commit message: assignment 7

File: body.urdf (robot description, URDF)
Before this commit: robot robot, 4 links, 3 joints
Links:
- added link 5, mass 1; collision box size=0.15738456030908277 0.3337268384711195 0.17346599743780305; visual box size=0.15738456030908277 0.3337268384711195 0.17346599743780305
- added link 6, mass 1; collision box size=1.048765667402233 1.1687671212833426 0.3356447484293533; visual box size=1.048765667402233 1.1687671212833426 0.3356447484293533
- added link 7, mass 1; collision box size=1.2061628238742597 1.192254274610946 0.5478718335460071; visual box size=1.2061628238742597 1.192254274610946 0.5478718335460071
- added link 8, mass 1; collision box size=1.884410037298442 0.8510806420637999 0.25898055277132676; visual box size=1.884410037298442 0.8510806420637999 0.25898055277132676
- added link 9, mass 1; collision box size=1.594249352408281 1.3036696330348025 0.5878322664553622; visual box size=1.594249352408281 1.3036696330348025 0.5878322664553622
- link 1: geometry collision box size=1.1461751177986281 0.9044457244864212 0.6905678287738731; visual box size=1.1461751177986281 0.9044457244864212 0.6905678287738731
- link 2: geometry collision box size=0.7869228015454138 0.3337268384711195 0.3469319948756061; visual box size=0.7869228015454138 0.3337268384711195 0.3469319948756061
- link 3: geometry collision box size=0.15738456030908277 0.3337268384711195 0.17346599743780305; visual box size=0.15738456030908277 0.3337268384711195 0.17346599743780305
- link 4: geometry collision box size=0.7869228015454138 0.3337268384711195 0.3469319948756061; visual box size=0.7869228015454138 0.3337268384711195 0.3469319948756061
Joints:
- removed joint 1_3
- removed joint 3_4
- added joint 1_4: type revolute, parent 1, child 4, origin xyz=0.0 -0.4522228622432106 1.8273580428065317 rpy=0 0 0, axis 1 1 0, limit lower=-3.14159 upper=3.14159 effort=0.0 velocity=0.0
- added joint 1_6: type revolute, parent 1, child 6, origin xyz=0.5730875588993141 0 2 rpy=0.20052398901919777 0 0.07023048521994799, axis 0 1 0, limit lower=-3.14159 upper=3.14159 effort=0.0 velocity=0.0
- added joint 2_3: type revolute, parent 2, child 3, origin xyz=0 0.3337268384711195 -0.08673299871890153 rpy=-45 0 0, axis 1 1 0, limit lower=-3.14159 upper=3.14159 effort=0.0 velocity=0.0
- added joint 4_5: type revolute, parent 4, child 5, origin xyz=0 -0.3337268384711195 -0.08673299871890153 rpy=45 0 0, axis 1 1 0, limit lower=-3.14159 upper=3.14159 effort=0.0 velocity=0.0
- added joint 6_7: type revolute, parent 6, child 7, origin xyz=1.048765667402233 0 0 rpy=0 0 0.016402351421724904, axis 0 1 0, limit lower=-3.14159 upper=3.14159 effort=0.0 velocity=0.0
- added joint 7_8: type revolute, parent 7, child 8, origin xyz=1.2061628238742597 0 0 rpy=0 0.1479099930739915 0.06028086801500576, axis 0 1 0, limit lower=-3.14159 upper=3.14159 effort=0.0 velocity=0.0
- added joint 8_9: type revolute, parent 8, child 9, origin xyz=1.884410037298442 0 0 rpy=0 0 0, axis 0 1 0, limit lower=-3.14159 upper=3.14159 effort=0.0 velocity=0.0
- joint 1_2: axis 0 1 0 -> 1 1 0; origin xyz=-0.35872688498709293 0 1 rpy=0 0 0 -> xyz=0.0 0.4522228622432106 1.8273580428065317 rpy=0 0 0
