Commit message: final prep

File: best1.urdf (robot description, URDF)
Before this commit: robot robot, 4 links, 3 joints
Links:
- added link 10, mass 1; collision box size=1.4715686666061312 0.7983114739411655 0.5958146288547794; visual box size=1.4715686666061312 0.7983114739411655 0.5958146288547794
- added link 11, mass 1; collision box size=1.8573097874080085 1.0524582116724508 0.3756277989076362; visual box size=1.8573097874080085 1.0524582116724508 0.3756277989076362
- added link 12, mass 1; collision box size=1.3332685670691757 0.5320391020442645 0.19367304155640844; visual box size=1.3332685670691757 0.5320391020442645 0.19367304155640844
- added link 13, mass 1; collision box size=1.3332685670691757 0.5320391020442645 0.19367304155640844; visual box size=1.3332685670691757 0.5320391020442645 0.19367304155640844
- added link 5, mass 1; collision box size=1.0699166946236416 0.44844311207175125 0.2982102450519535; visual box size=1.0699166946236416 0.44844311207175125 0.2982102450519535
- added link 6, mass 1; collision box size=1.0699166946236416 0.44844311207175125 0.2982102450519535; visual box size=1.0699166946236416 0.44844311207175125 0.2982102450519535
- added link 7, mass 1; collision box size=1.0699166946236416 0.44844311207175125 0.2982102450519535; visual box size=1.0699166946236416 0.44844311207175125 0.2982102450519535
- added link 8, mass 1; collision box size=1.2231832167407506 0.9145799030297643 0.5340343745433296; visual box size=1.2231832167407506 0.9145799030297643 0.5340343745433296
- added link 9, mass 1; collision box size=1.9957167748336653 1.0311035543585696 0.48453796470208954; visual box size=1.9957167748336653 1.0311035543585696 0.48453796470208954
- link 1: geometry collision box size=1.3468867510593867 1.4687290897826877 1.3872060036083016; visual box size=1.3468867510593867 1.4687290897826877 1.3872060036083016
- link 2: geometry collision box size=1.3976537361927084 0.6160344316030273 0.5953746369070513; visual box size=1.3976537361927084 0.6160344316030273 0.5953746369070513
- link 3: geometry collision box size=1.6529855242230023 1.11340412546957 0.5918013288350785; visual box size=1.6529855242230023 1.11340412546957 0.5918013288350785
- link 4: geometry collision box size=1.0699166946236416 0.44844311207175125 0.2982102450519535; visual box size=1.0699166946236416 0.44844311207175125 0.2982102450519535
Joints:
- removed joint 2_4
- added joint 10_11: type revolute, parent 10, child 11, origin xyz=1.4715686666061312 0 0 rpy=0 0 0, axis 0 1 0, limit lower=-3.14159 upper=3.14159 effort=0.0 velocity=0.0
- added joint 11_12: type revolute, parent 11, child 12, origin xyz=0.9286548937040042 0.5262291058362254 -0.09390694972690905 rpy=0 0 0, axis 1 1 0, limit lower=-3.14159 upper=3.14159 effort=0.0 velocity=0.0
- added joint 11_13: type revolute, parent 11, child 13, origin xyz=0.9286548937040042 -0.5262291058362254 -0.09390694972690905 rpy=0 0 0, axis 1 1 0, limit lower=-3.14159 upper=3.14159 effort=0.0 velocity=0.0
- added joint 2_10: type revolute, parent 2, child 10, origin xyz=1.3976537361927084 0 0 rpy=0 0 0, axis 0 1 0, limit lower=-3.14159 upper=3.14159 effort=0.0 velocity=0.0
- added joint 3_4: type revolute, parent 3, child 4, origin xyz=-0.8264927621115011 0.556702062734785 -0.14795033220876963 rpy=0 0 0, axis 1 1 0, limit lower=-3.14159 upper=3.14159 effort=0.0 velocity=0.0
- added joint 3_6: type revolute, parent 3, child 6, origin xyz=-0.8264927621115011 -0.556702062734785 -0.14795033220876963 rpy=0 0 0, axis 1 1 0, limit lower=-3.14159 upper=3.14159 effort=0.0 velocity=0.0
- added joint 3_8: type revolute, parent 3, child 8, origin xyz=-1.6529855242230023 0 0 rpy=0 0 0, axis 0 1 0, limit lower=-3.14159 upper=3.14159 effort=0.0 velocity=0.0
- added joint 4_5: type revolute, parent 4, child 5, origin xyz=0 0.44844311207175125 -0.07455256126298837 rpy=0 0 0, axis 1 1 0, limit lower=-3.14159 upper=3.14159 effort=0.0 velocity=0.0
- added joint 6_7: type revolute, parent 6, child 7, origin xyz=0 -0.44844311207175125 -0.07455256126298837 rpy=0 0 0, axis 1 1 0, limit lower=-3.14159 upper=3.14159 effort=0.0 velocity=0.0
- added joint 8_9: type revolute, parent 8, child 9, origin xyz=-1.2231832167407506 0 0 rpy=0 0 0, axis 0 1 0, limit lower=-3.14159 upper=3.14159 effort=0.0 velocity=0.0
- joint 1_2: origin xyz=0.7745302780565695 0 2 rpy=0 0 0 -> xyz=0.6734433755296934 0 2 rpy=0 0 0
- joint 1_3: origin xyz=-0.7745302780565695 0 2 rpy=0 0 0 -> xyz=-0.6734433755296934 0 2 rpy=0 0 0

File: best3.urdf (robot description, URDF)
Before this commit: robot robot, 8 links, 7 joints
Links:
- added link 10, mass 1; collision box size=1.6701005885047682 1.2155324172446744 0.2608247242036367; visual box size=1.6701005885047682 1.2155324172446744 0.2608247242036367
- added link 11, mass 1; collision box size=1.9337094542374902 1.0293596583124702 0.4904295398956208; visual box size=1.9337094542374902 1.0293596583124702 0.4904295398956208
- added link 9, mass 1; collision box size=1.7393550809894687 0.9430543847017234 0.38175459995781696; visual box size=1.7393550809894687 0.9430543847017234 0.38175459995781696
- link 1: geometry collision box size=1.0537466449639372 1.6317568953619581 0.8111463719892776; visual box size=1.0537466449639372 1.6317568953619581 0.8111463719892776
- link 2: geometry collision box size=1.9305501888392413 0.6154511334954655 0.497646080716015; visual box size=1.9305501888392413 0.6154511334954655 0.497646080716015
- link 3: geometry collision box size=1.921996299359665 0.4081655323445834 0.19963699242287727; visual box size=1.921996299359665 0.4081655323445834 0.19963699242287727
- link 4: geometry collision box size=1.921996299359665 0.4081655323445834 0.19963699242287727; visual box size=1.921996299359665 0.4081655323445834 0.19963699242287727
- link 5: geometry collision box size=1.4913614015788166 1.2236069456458476 0.2850258160685294; visual box size=1.4913614015788166 1.2236069456458476 0.2850258160685294
- link 6: geometry collision box size=1.5364260690575302 0.584574651370379 0.40396479292361404; visual box size=1.5364260690575302 0.584574651370379 0.40396479292361404
- link 7: geometry collision box size=1.0517798107962433 1.0615441815163162 0.40767102860065524; visual box size=1.0517798107962433 1.0615441815163162 0.40767102860065524
- link 8: geometry collision box size=1.0392196108896066 1.2675630264234927 0.42711310975052225; visual box size=1.0392196108896066 1.2675630264234927 0.42711310975052225
Joints:
- removed joint 1_6
- removed joint 3_4
- removed joint 3_5
- removed joint 3_8
- added joint 10_11: type revolute, parent 10, child 11, origin xyz=1.6701005885047682 0 0 rpy=0 0 0, axis 0 1 0, limit lower=-3.14159 upper=3.14159 effort=0.0 velocity=0.0
- added joint 1_5: type revolute, parent 1, child 5, origin xyz=0.5268733224819686 0 2 rpy=0 0 0, axis 0 1 0, limit lower=-3.14159 upper=3.14159 effort=0.0 velocity=0.0
- added joint 2_4: type revolute, parent 2, child 4, origin xyz=-0.9652750944196207 -0.30772556674773277 -0.12441152017900375 rpy=0 0 0, axis 1 1 0, limit lower=-3.14159 upper=3.14159 effort=0.0 velocity=0.0
- added joint 2_6: type revolute, parent 2, child 6, origin xyz=-1.9305501888392413 0 0 rpy=0 0 0, axis 0 1 0, limit lower=-3.14159 upper=3.14159 effort=0.0 velocity=0.0
- added joint 5_8: type revolute, parent 5, child 8, origin xyz=1.4913614015788166 0 0 rpy=0 0 0, axis 0 1 0, limit lower=-3.14159 upper=3.14159 effort=0.0 velocity=0.0
- added joint 8_9: type revolute, parent 8, child 9, origin xyz=1.0392196108896066 0 0 rpy=0 0 0, axis 0 1 0, limit lower=-3.14159 upper=3.14159 effort=0.0 velocity=0.0
- added joint 9_10: type revolute, parent 9, child 10, origin xyz=1.7393550809894687 0 0 rpy=0 0 0, axis 0 1 0, limit lower=-3.14159 upper=3.14159 effort=0.0 velocity=0.0
- joint 1_2: origin xyz=-0.8309751175009976 0 2 rpy=0 0 0 -> xyz=-0.5268733224819686 0 2 rpy=0 0 0
- joint 2_3: axis 0 1 0 -> 1 1 0; origin xyz=-1.834171444798332 0 0 rpy=0 0 0 -> xyz=-0.9652750944196207 0.30772556674773277 -0.12441152017900375 rpy=0 0 0
- joint 6_7: origin xyz=1.2469040634117443 0 0 rpy=0 0 0 -> xyz=-1.5364260690575302 0 0 rpy=0 0 0

File: best4.urdf (robot description, URDF)
Before this commit: robot robot, 5 links, 4 joints
Links:
- added link 10, mass 1; collision box size=1.2727284204876126 0.39874791858115494 0.17466135416941217; visual box size=1.2727284204876126 0.39874791858115494 0.17466135416941217
- added link 11, mass 1; collision box size=1.2727284204876126 0.39874791858115494 0.17466135416941217; visual box size=1.2727284204876126 0.39874791858115494 0.17466135416941217
- added link 12, mass 1; collision box size=1.2727284204876126 0.39874791858115494 0.17466135416941217; visual box size=1.2727284204876126 0.39874791858115494 0.17466135416941217
- added link 13, mass 1; collision box size=1.2727284204876126 0.39874791858115494 0.17466135416941217; visual box size=1.2727284204876126 0.39874791858115494 0.17466135416941217
- added link 14, mass 1; collision box size=1.1222043298525741 0.7820097158015967 0.48118129941686655; visual box size=1.1222043298525741 0.7820097158015967 0.48118129941686655
- added link 15, mass 1; collision box size=1.3318599169412473 0.4319718658314943 0.13212271180005705; visual box size=1.3318599169412473 0.4319718658314943 0.13212271180005705
- added link 16, mass 1; collision box size=1.3318599169412473 0.4319718658314943 0.13212271180005705; visual box size=1.3318599169412473 0.4319718658314943 0.13212271180005705
- added link 17, mass 1; collision box size=1.3890743824285914 0.5768476851359065 0.2735614915149603; visual box size=1.3890743824285914 0.5768476851359065 0.2735614915149603
- added link 18, mass 1; collision box size=1.9027670900575018 0.9221349954096535 0.5679584171102399; visual box size=1.9027670900575018 0.9221349954096535 0.5679584171102399
- added link 19, mass 1; collision box size=1.462101498261084 0.8866236516441894 0.2121183466512474; visual box size=1.462101498261084 0.8866236516441894 0.2121183466512474
- added link 20, mass 1; collision box size=1.828192877048362 0.703936058464631 0.44275322658344635; visual box size=1.828192877048362 0.703936058464631 0.44275322658344635
- added link 6, mass 1; collision box size=1.73970404485285 0.6653255196404317 0.35579367469435014; visual box size=1.73970404485285 0.6653255196404317 0.35579367469435014
- added link 7, mass 1; collision box size=1.0076166764137786 0.9970458346720683 0.4383773768474517; visual box size=1.0076166764137786 0.9970458346720683 0.4383773768474517
- added link 8, mass 1; collision box size=1.1778101682445152 0.9824263983133119 0.5122176183978379; visual box size=1.1778101682445152 0.9824263983133119 0.5122176183978379
- added link 9, mass 1; collision box size=1.8329522043428192 1.0808706644694646 0.5586913389114221; visual box size=1.8329522043428192 1.0808706644694646 0.5586913389114221
- link 1: geometry collision box size=1.6377298936934426 0.9315181521757802 0.8853251882384129; visual box size=1.6377298936934426 0.9315181521757802 0.8853251882384129
- link 2: geometry collision box size=1.6874456500954875 1.0556336185288628 0.5079203359080494; visual box size=1.6874456500954875 1.0556336185288628 0.5079203359080494
- link 3: geometry collision box size=1.6574060415205016 0.7270859631481978 0.4996841902094703; visual box size=1.6574060415205016 0.7270859631481978 0.4996841902094703
- link 4: geometry collision box size=1.2570920018478315 1.2476316566634216 0.5158719540031944; visual box size=1.2570920018478315 1.2476316566634216 0.5158719540031944
- link 5: geometry collision box size=1.6541751245147138 0.9979296814169427 0.36793913180671495; visual box size=1.6541751245147138 0.9979296814169427 0.36793913180671495
Joints:
- removed joint 2_3
- removed joint 3_4
- added joint 10_11: type revolute, parent 10, child 11, origin xyz=0 0.39874791858115494 -0.04366533854235304 rpy=0 0 0, axis 1 1 0, limit lower=-3.14159 upper=3.14159 effort=0.0 velocity=0.0
- added joint 12_13: type revolute, parent 12, child 13, origin xyz=0 -0.39874791858115494 -0.04366533854235304 rpy=0 0 0, axis 1 1 0, limit lower=-3.14159 upper=3.14159 effort=0.0 velocity=0.0
- added joint 14_15: type revolute, parent 14, child 15, origin xyz=0.5611021649262871 0.39100485790079836 -0.12029532485421664 rpy=0 0 0, axis 1 1 0, limit lower=-3.14159 upper=3.14159 effort=0.0 velocity=0.0
- added joint 14_16: type revolute, parent 14, child 16, origin xyz=0.5611021649262871 -0.39100485790079836 -0.12029532485421664 rpy=0 0 0, axis 1 1 0, limit lower=-3.14159 upper=3.14159 effort=0.0 velocity=0.0
- added joint 14_17: type revolute, parent 14, child 17, origin xyz=1.1222043298525741 0 0 rpy=0 0 0, axis 0 1 0, limit lower=-3.14159 upper=3.14159 effort=0.0 velocity=0.0
- added joint 17_18: type revolute, parent 17, child 18, origin xyz=1.3890743824285914 0 0 rpy=0 0 0, axis 0 1 0, limit lower=-3.14159 upper=3.14159 effort=0.0 velocity=0.0
- added joint 18_19: type revolute, parent 18, child 19, origin xyz=1.9027670900575018 0 0 rpy=0 0 0, axis 0 1 0, limit lower=-3.14159 upper=3.14159 effort=0.0 velocity=0.0
- added joint 1_3: type revolute, parent 1, child 3, origin xyz=-0.8188649468467213 0 2 rpy=0 0 0, axis 0 1 0, limit lower=-3.14159 upper=3.14159 effort=0.0 velocity=0.0
- added joint 2_4: type revolute, parent 2, child 4, origin xyz=1.6874456500954875 0 0 rpy=0 0 0, axis 0 1 0, limit lower=-3.14159 upper=3.14159 effort=0.0 velocity=0.0
- added joint 4_6: type revolute, parent 4, child 6, origin xyz=1.2570920018478315 0 0 rpy=0 0 0, axis 0 1 0, limit lower=-3.14159 upper=3.14159 effort=0.0 velocity=0.0
- added joint 5_7: type revolute, parent 5, child 7, origin xyz=-1.6541751245147138 0 0 rpy=0 0 0, axis 0 1 0, limit lower=-3.14159 upper=3.14159 effort=0.0 velocity=0.0
- added joint 6_9: type revolute, parent 6, child 9, origin xyz=1.73970404485285 0 0 rpy=0 0 0, axis 0 1 0, limit lower=-3.14159 upper=3.14159 effort=0.0 velocity=0.0
- added joint 7_8: type revolute, parent 7, child 8, origin xyz=-1.0076166764137786 0 0 rpy=0 0 0, axis 0 1 0, limit lower=-3.14159 upper=3.14159 effort=0.0 velocity=0.0
- added joint 8_20: type revolute, parent 8, child 20, origin xyz=-1.1778101682445152 0 0 rpy=0 0 0, axis 0 1 0, limit lower=-3.14159 upper=3.14159 effort=0.0 velocity=0.0
- added joint 9_10: type revolute, parent 9, child 10, origin xyz=0.9164761021714096 0.5404353322347323 -0.13967283472785552 rpy=0 0 0, axis 1 1 0, limit lower=-3.14159 upper=3.14159 effort=0.0 velocity=0.0
- added joint 9_12: type revolute, parent 9, child 12, origin xyz=0.9164761021714096 -0.5404353322347323 -0.13967283472785552 rpy=0 0 0, axis 1 1 0, limit lower=-3.14159 upper=3.14159 effort=0.0 velocity=0.0
- added joint 9_14: type revolute, parent 9, child 14, origin xyz=1.8329522043428192 0 0 rpy=0 0 0, axis 0 1 0, limit lower=-3.14159 upper=3.14159 effort=0.0 velocity=0.0
- joint 1_2: origin xyz=-0.9946508487550862 0 2 rpy=0 0 0 -> xyz=0.8188649468467213 0 2 rpy=0 0 0
- joint 3_5: axis 1 1 0 -> 0 1 0; origin xyz=-0.9332628339011111 -0.3498103934170069 -0.06541353189260608 rpy=0 0 0 -> xyz=-1.6574060415205016 0 0 rpy=0 0 0

File: best5.urdf (robot description, URDF)
Before this commit: robot robot, 6 links, 5 joints
Links:
- removed link 5
- removed link 6
- removed link 7
- added link 4, mass 1; collision box size=1.8340039036183042 0.9791238170967902 0.2541198687610006; visual box size=1.8340039036183042 0.9791238170967902 0.2541198687610006
- link 1: geometry collision box size=1.6632706384743012 1.4311193334160057 0.9547409147594323; visual box size=1.6632706384743012 1.4311193334160057 0.9547409147594323
- link 2: geometry collision box size=1.2851808426272175 0.994860534775835 0.408230335467077; visual box size=1.2851808426272175 0.994860534775835 0.408230335467077
- link 3: geometry collision box size=1.5738445671356789 0.5703746191768697 0.47832813607553143; visual box size=1.5738445671356789 0.5703746191768697 0.47832813607553143
Joints:
- removed joint 2_5
- removed joint 5_6
- removed joint 5_7
- added joint 2_4: type revolute, parent 2, child 4, origin xyz=-1.2851808426272175 0 0 rpy=0 0 0, axis 0 1 0, limit lower=-3.14159 upper=3.14159 effort=0.0 velocity=0.0
- joint 1_2: origin xyz=-0.8558297948056166 0 2 rpy=0 0 0 -> xyz=-0.8316353192371506 0 2 rpy=0 0 0
- joint 1_3: origin xyz=0.8558297948056166 0 2 rpy=0 0 0 -> xyz=0.8316353192371506 0 2 rpy=0 0 0

File: body5007.urdf (robot description, URDF)
Before this commit: robot robot, 10 links, 9 joints
Links:
- link 1: geometry collision box size=1.0678631343578746 1.1463347974848481 1.4613124315551445; visual box size=1.0678631343578746 1.1463347974848481 1.4613124315551445
- link 10: geometry collision box size=1.0533773230856256 0.558499088737178 0.13657323805441002; visual box size=1.0533773230856256 0.558499088737178 0.13657323805441002
- link 2: geometry collision box size=1.0147927621608086 0.7960844883011403 0.7992226138411569; visual box size=1.0147927621608086 0.7960844883011403 0.7992226138411569
- link 3: geometry collision box size=1.0147927621608086 0.7960844883011403 0.7992226138411569; visual box size=1.0147927621608086 0.7960844883011403 0.7992226138411569
- link 4: geometry collision box size=1.0147927621608086 0.7960844883011403 0.7992226138411569; visual box size=1.0147927621608086 0.7960844883011403 0.7992226138411569
- link 5: geometry collision box size=1.0147927621608086 0.7960844883011403 0.7992226138411569; visual box size=1.0147927621608086 0.7960844883011403 0.7992226138411569
- link 6: geometry collision box size=1.5505851730076525 0.8721469829956152 0.45223060138285637; visual box size=1.5505851730076525 0.8721469829956152 0.45223060138285637
- link 7: geometry collision box size=1.0533773230856256 0.558499088737178 0.13657323805441002; visual box size=1.0533773230856256 0.558499088737178 0.13657323805441002
- link 8: geometry collision box size=1.0533773230856256 0.558499088737178 0.13657323805441002; visual box size=1.0533773230856256 0.558499088737178 0.13657323805441002
- link 9: geometry collision box size=1.0533773230856256 0.558499088737178 0.13657323805441002; visual box size=1.0533773230856256 0.558499088737178 0.13657323805441002
Joints:
- removed joint 1_8
- removed joint 3_4
- removed joint 3_6
- removed joint 3_9
- removed joint 8_10
- added joint 1_4: type revolute, parent 1, child 4, origin xyz=0.0 -0.5731673987424241 1.6346718921112138 rpy=0 0 0, axis 1 1 0, limit lower=-3.14159 upper=3.14159 effort=0.0 velocity=0.0
- added joint 1_6: type revolute, parent 1, child 6, origin xyz=-0.5339315671789373 0 2 rpy=0 0 0, axis 0 1 0, limit lower=-3.14159 upper=3.14159 effort=0.0 velocity=0.0
- added joint 6_9: type revolute, parent 6, child 9, origin xyz=-0.7752925865038263 -0.4360734914978076 -0.11305765034571409 rpy=0 0 0, axis 1 1 0, limit lower=-3.14159 upper=3.14159 effort=0.0 velocity=0.0
- added joint 7_8: type revolute, parent 7, child 8, origin xyz=0 0.558499088737178 -0.034143309513602504 rpy=0 0 0, axis 1 1 0, limit lower=-3.14159 upper=3.14159 effort=0.0 velocity=0.0
- added joint 9_10: type revolute, parent 9, child 10, origin xyz=0 -0.558499088737178 -0.034143309513602504 rpy=0 0 0, axis 1 1 0, limit lower=-3.14159 upper=3.14159 effort=0.0 velocity=0.0
- joint 1_2: axis 0 1 0 -> 1 1 0; origin xyz=-0.8519625687814558 0 2 rpy=0 0 0 -> xyz=0.0 0.5731673987424241 1.6346718921112138 rpy=0 0 0
- joint 2_3: axis 0 1 0 -> 1 1 0; origin xyz=-1.7101996074265777 0 0 rpy=0 0 0 -> xyz=0 0.7960844883011403 -0.19980565346028922 rpy=0 0 0
- joint 4_5: origin xyz=0 0.39536396679258895 -0.0771228199101844 rpy=0 0 0 -> xyz=0 -0.7960844883011403 -0.19980565346028922 rpy=0 0 0
- joint 6_7: origin xyz=0 -0.39536396679258895 -0.0771228199101844 rpy=0 0 0 -> xyz=-0.7752925865038263 0.4360734914978076 -0.11305765034571409 rpy=0 0 0
